File: space_shuttle_SAO/space_shuttle_SAO.kicad_sch (KiCad schematic)
At the start: 5 parts, among them J1 SAO_1.69, SW1 SW_SPDT

Commit message: weekend updates to Wright Stuff
Parts:
- BT1: MPN (none) -> 3034
- D1: MPN (none) -> XZMYK45WT-9
- R1: MPN (none) -> RC1206FR-07330RL
- SW1: MPN (none) -> SWITCH SLIDE DPDT 300MA 6V
