File: Badge/WrightSpace/WrightSpace.kicad_sch (KiCad schematic)
At the start: 49 parts, among them J1 Conn_02x03_Counter_Clockwise, SW1 SW_SPDT, SW2 SW_SPDT, U1 ESP32-S2-SOLO

Commit message: transitor additions for LEDs
Parts:
- removed R1, R10, R2, R8, R9: 30, Resistor_SMD:R_0805_2012Metric, symbol Device:R
- added Q1, Q2, Q3, Q4, Q5, Q6: BC817, Package_TO_SOT_SMD:SOT-23, symbol Transistor_BJT:BC817
- added R13: 30, Resistor_SMD:R_0805_2012Metric, symbol Device:R
- added R6: 1K, Resistor_SMD:R_0805_2012Metric, symbol Device:R
- C4: renamed from C2; value 10uF -> 1uF
- C5: renamed from C3; value 1uF -> 10uF
- D1, D2, D3, D4, D5: MPN XZMDKCBDDG45S-9 -> (none)
- R11: value 30 -> 150; MPN RC0805FR-0730RL -> RC0805JR-07150RL
- R12: value 150 -> 30; MPN RC0805JR-07150RL -> RC0805FR-0730RL
- R14, R15, R16: value 150 -> 1K; MPN RC0805JR-07150RL -> RNCP0805FTD1K00
- R4, R5: value 30 -> 1K; MPN RC0805FR-0730RL -> RNCP0805FTD1K00
- R7: renamed from R6; value 5K -> 4.7K
- renumbered C4 to C1, C5 to C2, C1 to C3, J2 to J1, J1 to J2, R13 to R1, R24 to R10, R7 to R2, R25 to R8, R23 to R9, SW2 to SW1, SW1 to SW2, U2 to U1, U1 to U2
Connections:
- net GND: now also Q1.2 (E), Q2.2 (E), Q3.2 (E), Q4.2 (E), Q5.2 (E), Q6.2 (E)
- net LED1_B: now also R5.1
- net LED1_G: now also R6.1; no longer R2.1
- net LED1_R: now also R4.1; no longer R1.1, R12.1
- net LED2_B: now also R15.1; no longer R3.1, R4.1, R5.1
- net LED2_G: now also R16.1; no longer R11.1
- net LED2_R: no longer R15.1, R16.1
- net at D1.3 (B), R2.2: now also D2.3 (B)
- net at D2.4 (G): now also D1.4 (G), R3.2
- net at D4.3 (B): now also D3.3 (B), D5.3 (B), R12.2
- net at D3.1 (R): now also D4.1 (R), D5.1 (R), R11.1; no longer R14.2
- net at R16.2: now also Q6.1 (B); no longer D5.1 (R)
- net at D3.4 (G): now also D4.4 (G), D5.4 (G), R13.2; no longer R3.2
- net at D1.1 (R): now also D2.1 (R), R1.1; no longer R12.2
- net at R15.2: now also Q5.1 (B); no longer D4.1 (R)
- net at R4.2: now also Q1.1 (B); no longer D4.4 (B)
- net at R1.2: now also Q1.3 (C); no longer D2.1 (R)
- net at R11.2: now also Q4.3 (C); no longer D5.3 (G)
- net at R5.2: now also Q2.1 (B); no longer D5.4 (B)
- new net: Q2.3 (C), R2.1
- new net: Q3.1 (B), R6.2
- new net: Q3.3 (C), R3.1
- new net: Q6.3 (C), R13.1
- new net: Q4.1 (B), R14.2
- new net: Q5.3 (C), R12.1
Other:
- note added: "Alien LEDs"
- note added: "Satellite LEDs"
- note added: "Star LEDs"
- note removed: "LEDs"
- moved on the sheet: D10, D11, D6, D7, D8, D9, R10, R17, R18, R19, R20, R21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

Commit message: v04 of Wright Flyer
Parts:
- added D12, D13, D14: SunLED_RGB_ReverseMount, sunled:XZMDKCBDDG45S-9, symbol LED:SunLED_RGB_ReverseMount
- added Q7, Q8, Q9: BC817, Package_TO_SOT_SMD:SOT-23, symbol Transistor_BJT:BC817
- added R23, R25, R27: 1K, Resistor_SMD:R_0805_2012Metric, symbol Device:R
- added R24, R29, R34: 150, Resistor_SMD:R_0805_2012Metric, symbol Device:R
- added R30, R31, R32, R33, R35, R36: 30, Resistor_SMD:R_0805_2012Metric, symbol Device:R
Connections:
- net GND: now also Q7.2 (E), Q8.2 (E), Q9.2 (E)
- net LED2_B: now also R25.1
- net LED2_G: now also R27.1
- net LED2_R: now also R23.1
- net VDD33: now also D12.2 (A), D13.2 (A), D14.2 (A)
- new net: Q9.3 (C), R31.1, R33.1, R36.1
- new net: D13.4 (G), R33.2
- new net: Q8.1 (B), R25.2
- new net: Q8.3 (C), R30.1, R32.1, R35.1
- new net: Q7.1 (B), R23.2
- new net: Q7.3 (C), R24.2, R29.2, R34.2
- new net: D14.3 (B), R35.2
- new net: D14.1 (R), R34.1
- new net: D14.4 (G), R36.2
- new net: Q9.1 (B), R27.2
- new net: D12.1 (R), R29.1
- new net: D12.3 (B), R30.2
- new net: D12.4 (G), R31.2
- new net: D13.1 (R), R24.1
- new net: D13.3 (B), R32.2

Commit message: v02 up for final review
Parts:
- removed D13, D14, D3: SunLED_RGB_ReverseMount, sunled:XZMDKCBDDG45S-9, symbol LED:SunLED_RGB_ReverseMount
- removed Q4, Q5, Q6: BC817, Package_TO_SOT_SMD:SOT-23, symbol Transistor_BJT:BC817
- removed R11, R34: 150, Resistor_SMD:R_0805_2012Metric, symbol Device:R
- removed R12, R13, R32, R33, R36: 30, Resistor_SMD:R_0805_2012Metric, symbol Device:R
- removed R14, R15, R16: 1K, Resistor_SMD:R_0805_2012Metric, symbol Device:R
- added D13: LED, aerospace_badge:led_in-s124ar, symbol Device:LED
- added D6: SunLED_RGB_ReverseMount, sunled:XZMDKCBDDG45S-9, symbol LED:SunLED_RGB_ReverseMount
- added R17, R20, R23: 150, Resistor_SMD:R_0805_2012Metric, symbol Device:R
- added R18, R19, R21, R22, R25: 30, Resistor_SMD:R_0805_2012Metric, symbol Device:R
- added R7, R8, R9: 1K, Resistor_SMD:R_0805_2012Metric, symbol Device:R
- R24: value 150 -> 30; MPN RC0805JR-07150RL -> RC0805FR-0730RL
- R35: value 30 -> 330; footprint Resistor_SMD:R_0805_2012Metric -> Resistor_SMD:R_0805_2012Metric_Pad1.20x1.40mm_HandSolder; MPN RC0805FR-0730RL -> (none)
- R4: value 1K -> 150; MPN RNCP0805FTD1K00 -> RC0805JR-07150RL
- R5, R6: value 1K -> 30; MPN RNCP0805FTD1K00 -> RC0805FR-0730RL
- renumbered D9 to D10, D10 to D11, D11 to D12, D12 to D3, D6 to D7, D7 to D8, D8 to D9, J2 to J1, J3 to J2, J1 to J3, Q7 to Q4, Q8 to Q5, Q9 to Q6, R7 to R10, R8 to R11, R9 to R12, R10 to R13, R29 to R14, R30 to R15, R31 to R16, R23 to R26, R25 to R27, R27 to R28, R17 to R29, R18 to R30, R19 to R31, R20 to R32, R21 to R33, R22 to R34
Connections:
- net GND: now also R35.2
- net LED1_B: now also R8.1; no longer R5.1
- net LED1_G: now also R9.1; no longer R6.1
- net LED1_R: now also R7.1; no longer R4.1
- net VDD33: now also D6.2 (A)
- net at D5.1 (R): now also R20.1; no longer D4.1 (R)
- net at D5.3 (B): now also R21.2; no longer D4.3 (B)
- net at D5.4 (G): now also R22.2; no longer D4.4 (G)
- net at Q2.3 (C), R2.1: now also R5.1
- net at D1.3 (B), R2.2: no longer D2.3 (B)
- net at R6.2: now also D2.4 (G); no longer Q3.1 (B)
- net at Q3.3 (C), R3.1: now also R6.1
- net at Q6.3 (C), R16.1: now also R19.1, R22.1, R25.1
- net at Q5.3 (C), R15.1: now also R24.1, R18.1, R21.1; no longer R35.1
- net at Q4.3 (C), R14.2: now also R17.2, R20.2, R23.2; no longer R24.2
- net at Q1.1 (B): now also R7.2; no longer R4.2
- net at Q1.3 (C), R1.2: now also R4.2
- net at D1.4 (G), R3.2: no longer D2.4 (G)
- net at Q2.1 (B): now also R8.2; no longer R5.2
- net at D1.1 (R), R1.1: no longer D2.1 (R)
- net LED7: now reaches U2.29 (SPIIO7/GPIO36/FSPICLK)
- net LED7: now also D13.2 (A)
- new net: D13.1 (K), R35.1
- new net: Q3.1 (B), R9.2
- new net: D2.1 (R), R4.1
- new net: D2.3 (B), R5.2
- new net: D6.1 (R), R23.1
- new net: D4.1 (R), R17.1
- new net: D6.3 (B), R24.2
- new net: D4.4 (G), R19.2
- new net: D6.4 (G), R25.2
- new net: D4.3 (B), R18.2
- no-connect marks 15 -> 14
Other:
- note added: "Alien LED"
- note removed: "Alien LEDs"
- moved on the sheet: D10, D11, D12, D3, D7, D8, D9, J1, J2, J3, Q4, Q5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
